Commit message: Adding MoveIt Package and continuous_move.py script for robot's movents Signe-off-by: Luca Inghilterra E-mail: 271539@studenti.unimore.it

File: src/pastabot_pkg/urdf/gofa_arm_urdf_toolfixed.urdf (robot description, URDF)
Before this commit: robot gofa_arm_urdf, 15 links, 14 joints
Links:
- link link01_rev1: mass None -> 0.1
- link link02_rev2: mass None -> 0.1
- link link03_rev3: mass None -> 0.1
- link link04_rev4: mass None -> 0.1
- link link05_rev5: mass None -> 0.1
- link link06_rev6: mass None -> 0.1

Commit message: Project's Update Signed-off by: Luca Inghilterra Email: 271539@studenti.unimore.it

File: src/pastabot_pkg/urdf/gofa_arm_urdf_toolfixed.urdf (robot description, URDF)
Before this commit: robot gofa_arm_urdf, 15 links, 14 joints
Joints:
- joint jnt2_DH: limit lower=-3.14159 upper=3.14159 effort=1000.0 velocity=50.0 -> lower=-1.5708 upper=1.5708 effort=1000.0 velocity=50.0
- joint jnt2_rev: limit lower=-3.14159 upper=3.14159 effort=1000.0 velocity=50.0 -> lower=-1.5708 upper=1.5708 effort=1000.0 velocity=50.0
- joint jnt3_DH: limit lower=-3.14159 upper=3.14159 effort=1000.0 velocity=50.0 -> lower=-1.5708 upper=1.5708 effort=1000.0 velocity=50.0
- joint jnt3_rev: limit lower=-3.14159 upper=3.14159 effort=1000.0 velocity=50.0 -> lower=-1.5708 upper=1.5708 effort=1000.0 velocity=50.0
